File: internship.kicad_pcb (KiCad board)
At the start: 2 copper layers, 100 x 100 mm, 83 parts, among them J1 3.7V_LIPO, J2 USB_C_16P, J3 RC_RECEIVER, J4 M1_MOTOR, J5 M2_MOTOR, J6 M3_MOTOR, J7 M4_MOTOR, J8 GPS_MODULE, J9 I2C_COMPASS, Q1 AO3400A, Q2 AO3400A, Q3 AO3400A, Q4 AO3400A, Q5 AO3400A, Q6 AO3400A, SW1 RESET, SW2 BOOT, SW3 PWR_SW, U1 ESP32-S3-WROOM-1, U2 ICM-42688-P, U4 TP4056, U5 AP2112K-3.3, U6 BMP280

Commit message: Add secondary MPU-6050 IMU (U3 + C4, C5, C8) on B.Cu and update Gerbers/Manufacturing Pack
Parts:
- added C4: 100nF, C_0603_1608Metric, B.Cu at (168.5, 96.5)
- added C5: 100nF, C_0603_1608Metric, B.Cu at (168.5, 98.2)
- added C8: 100nF, C_0603_1608Metric, B.Cu at (162.5, 91.2)
- added U3: MPU-6050, InvenSense_QFN-24_4x4mm_P0.5mm, B.Cu at (164.0, 95.0)
Routing:
- net +3V3: track 152.8 -> 182.9 mm, vias 6 -> 7
- net /ESP_SDA: track 23.4 -> 46.3 mm, vias 1 -> 6
- net /ESP_SCL: track 16.5 -> 38.5 mm, vias 1 -> 6
- net GND: track 325.4 -> 335.8 mm, vias 3 -> 7
- net Net-(U3-REGOUT): track 0.00 -> 5.18 mm
- net Net-(U3-CPOUT): track 0.00 -> 3.42 mm
Other:
- board text removed: "ESP32-S3 MICRO DRONE"
